Commit message: fixed scout urdf

File: scout_ros/scout_description/urdf/scout_v2.xacro (robot description, xacro)
@@ -3,6 +3,5 @@
     <xacro:arg name="botname" default=""/>
     <xacro:include filename="$(find scout_description)/urdf/common_properties.xacro" />
-    <xacro:include filename="$(find scout_description)/urdf/scout/scout_v2.gazebo.xacro" />
-    <xacro:arg name="robot_namespace" default="/" />
+    <xacro:include filename="$(find scout_description)/urdf/scout_v2.gazebo.xacro" />
     <xacro:include filename="$(find scout_description)/urdf/scout_wheel_type1.xacro" />
     <xacro:include filename="$(find scout_description)/urdf/scout_wheel_type2.xacro" />
@@ -40,5 +39,5 @@
     </link>
     <link name="base_footprint"/>
-    <joint name="base_footprint_joint" type="fixed">
+    <joint name="base_link_joint" type="fixed">
         <origin xyz="0 0 ${wheel_radius - wheel_vertical_offset}" rpy="0 0 0" />
         <parent link="base_footprint" />
@@ -66,5 +65,5 @@
         <origin xyz="0 0 0.0" rpy="0 0 0"/>
         <geometry>
-          <mesh filename="package://scout_description/meshes/scout/hokuyo.dae"/>
+          <mesh filename="package://scout_description/meshes/hokuyo.dae"/>
         </geometry>
         <material name="dark"/>
@@ -88,5 +87,5 @@
     <!-- motor 1 and 2 (left side) are mechanically installed in a reversed direction -->
     <xacro:scout_wheel_type1 wheel_prefix="front_right">
-        <origin xyz="${wheelbase/2} ${-track/2} ${wheel_vertical_offset}" rpy="3.14 0 0" />
+        <origin xyz="${wheelbase/2} ${-track/2} ${wheel_vertical_offset}" rpy="0 0 0" />
     </xacro:scout_wheel_type1>
     <xacro:scout_wheel_type2 wheel_prefix="front_left">
@@ -97,5 +96,5 @@
     </xacro:scout_wheel_type1>
     <xacro:scout_wheel_type2 wheel_prefix="rear_right">
-        <origin xyz="${-wheelbase/2} ${-track/2} ${wheel_vertical_offset}" rpy="3.14 0 0" />
+        <origin xyz="${-wheelbase/2} ${-track/2} ${wheel_vertical_offset}" rpy="0 0 0" />
     </xacro:scout_wheel_type2>
 </robot>

File: scout_ros/scout_description/urdf/scout_wheel_type1.xacro (robot description, xacro)
@@ -48,5 +48,5 @@
             <child link="${wheel_prefix}_wheel_link"/>
             <xacro:insert_block name="joint_pose"/>
-            <axis xyz="0 -1 0" rpy="0 0 0" />
+            <axis xyz="0 1 0" rpy="0 0 0" />
         </joint>
         <transmission name="${wheel_prefix}_wheel_trans">
@@ -60,4 +60,3 @@
         </transmission>
     </xacro:macro>
-    </xacro:macro>
 </robot>

File: scout_ros/scout_description/urdf/scout_wheel_type2.xacro (robot description, xacro)
@@ -48,5 +48,5 @@
             <child link="${wheel_prefix}_wheel_link"/>
             <xacro:insert_block name="joint_pose"/>
-            <axis xyz="0 -1 0" rpy="0 0 0" />
+            <axis xyz="0 1 0" rpy="0 0 0" />
         </joint>
         <transmission name="${wheel_prefix}_wheel_trans">
